Commit message: tricycle sim

File: description/03_tricycle_drive.xacro (robot description, xacro)
@@ -1,16 +1,4 @@
 <?xml version="1.0"?>
-<robot name="tricycle_drive" xmlns:xacro="http://ros.org/wiki/xacro">
-  <material name="Black">
-    <color rgba="0 0 0 1" />
-  </material>
-  <material name="Grey">
-    <color rgba="0.8 0.8 0.8 1" />
-  </material>
-  <material name="Orange">
-    <color rgba="1 0.6 0 1" />
-  </material>
-  <material name="White">
-    <color rgba="1 1 1 1" />
-  </material>
+<robot xmlns:xacro="http://ros.org/wiki/xacro">
   <link name="base_link" />
   <!-- Chassis -->
@@ -135,22 +123,3 @@
     <axis xyz="0 0 1" />
   </joint>
-  <ros2_control name="GazeboSystem" type="system">
-    <hardware>
-      <plugin>gazebo_ros2_control/GazeboSystem</plugin>
-    </hardware>
-    <joint name="steering_joint">
-      <command_interface name="position" />
-      <state_interface name="position" />
-    </joint>
-    <joint name="traction_joint">
-      <command_interface name="velocity" />
-      <state_interface name="velocity" />
-      <state_interface name="position" />
-    </joint>
-  </ros2_control>
-  <gazebo>
-    <plugin filename="libgazebo_ros2_control.so" name="gazebo_ros2_control">
-      <parameters>$(find f112th_sim_2401_fox)/config/tricycle_drive_controller.yaml</parameters>
-    </plugin>
-  </gazebo>
 </robot>

Commit message: tricycle 2 bicycle w problems

File: description/03_tricycle_drive.xacro (robot description, xacro)
@@ -43,5 +43,5 @@
     <collision>
       <geometry>
-        <cylinder length="${wheel_len}" radius="${wheel_radius}" />
+        <sphere radius="${wheel_radius}" />
       </geometry>
     </collision>
@@ -58,4 +58,5 @@
   </link>
   <joint name="left_wheel_joint" type="continuous">
+    <mimic joint="left_traction_joint"/>
     <origin xyz="-${base_lx/2} ${base_ly/2+wheel_len/2} -${base_lz/2}" rpy="-1.57 0 0" />
     <parent link="chassis" />
@@ -68,5 +69,5 @@
     <collision>
       <geometry>
-        <cylinder length="${wheel_len}" radius="${wheel_radius}" />
+        <sphere radius="${wheel_radius}" />
       </geometry>
     </collision>
@@ -83,4 +84,5 @@
   </link>
   <joint name="right_wheel_joint" type="continuous">
+    <mimic joint="left_traction_joint"/>
     <origin xyz="-${base_lx/2} -${base_ly/2+wheel_len/2} -${base_lz/2}" rpy="-1.57 0 0" />
     <parent link="chassis" />
@@ -103,9 +105,10 @@
     </inertial>
   </link>
-  <joint name="left_steering_joint" type="continuous">
+  <joint name="left_steering_joint" type="revolute">
     <origin xyz="${base_lx/2} ${base_ly/2+wheel_len/2} -${base_lz/2}" rpy="0 0 0" />
     <parent link="chassis" />
     <child link="left_steering_link" />
     <axis xyz="0 0 1" />
+    <limit effort="100.0" lower="-0.785398" upper="0.785398" velocity="0.1"/>
   </joint>
   <!-- traction wheel link -->
@@ -124,5 +127,5 @@
     <collision>
       <geometry>
-        <cylinder length="${wheel_len}" radius="${wheel_radius}" />
+        <sphere radius="${wheel_radius}" />
       </geometry>
     </collision>
@@ -149,5 +152,5 @@
     </inertial>
   </link>
-  <joint name="right_steering_joint" type="continuous">
+  <joint name="right_steering_joint" type="revolute">
     <mimic joint="left_steering_joint"/>
     <origin xyz="${base_lx/2} -${base_ly/2+wheel_len/2} -${base_lz/2}" rpy="0 0 0" />
@@ -155,4 +158,5 @@
     <child link="right_steering_link" />
     <axis xyz="0 0 1" />
+    <limit effort="100.0" lower="-0.785398" upper="0.785398" velocity="0.1"/>
   </joint>
   <!-- traction wheel link -->
@@ -171,5 +175,5 @@
     <collision>
       <geometry>
-        <cylinder length="${wheel_len}" radius="${wheel_radius}" />
+        <sphere radius="${wheel_radius}" />
       </geometry>
     </collision>

File: description/04_ros2_control.xacro (robot description, xacro)
@@ -6,8 +6,12 @@
     </hardware>
     <joint name="left_steering_joint">
+        <param name="min">-0.785</param>
+        <param name="max">0.785</param>
       <command_interface name="position" />
       <state_interface name="position" />
     </joint>
     <joint name="right_steering_joint">
+        <param name="min">-0.785</param>
+        <param name="max">0.785</param>
       <param name="mimic">left_steering_joint</param>
       <param name="multiplier">1</param>
