Commit message: bicycle try

File: description/01_properties.xacro (robot description, xacro)
@@ -1,4 +1,14 @@
 <?xml version="1.0"?>
 <robot xmlns:xacro="http://www.ros.org/wiki/xacro">
+  <!-- Constants for robot dimensions -->
+  <xacro:property name="PI" value="3.1415926535897931"/>
+  <xacro:property name="cm2m" value="0.01" /> <!-- arbitrary value for base mass -->
+  <xacro:property name="base_lx" value="${35.6*cm2m}" />
+  <xacro:property name="base_ly" value="${20.8*cm2m}" />
+  <xacro:property name="base_lz" value="${8.0*cm2m}" />
+  <xacro:property name="base_mass" value="2.0" />
+  <xacro:property name="wheel_mass" value=".25" /> <!-- arbitrary value for wheel mass -->
+  <xacro:property name="wheel_len" value="${3*cm2m}" />
+  <xacro:property name="wheel_radius" value="${3.5*cm2m}" />
   <material name="Black">
     <color rgba="0 0 0 1" />

File: description/03_tricycle_drive.xacro (robot description, xacro)
@@ -2,14 +2,4 @@
 <robot xmlns:xacro="http://ros.org/wiki/xacro">
   <xacro:include filename="02_inertia_macro.xacro"/>
-  <!-- Constants for robot dimensions -->
-  <xacro:property name="PI" value="3.1415926535897931"/>
-  <xacro:property name="cm2m" value="0.01" /> <!-- arbitrary value for base mass -->
-  <xacro:property name="base_lx" value="${35.6*cm2m}" />
-  <xacro:property name="base_ly" value="${20.8*cm2m}" />
-  <xacro:property name="base_lz" value="${11.0*cm2m}" />
-  <xacro:property name="base_mass" value="2.0" />
-  <xacro:property name="wheel_mass" value=".25" /> <!-- arbitrary value for wheel mass -->
-  <xacro:property name="wheel_len" value="${3*cm2m}" />
-  <xacro:property name="wheel_radius" value="${3.5*cm2m}" />
   <link name="base_link" />
   <!-- Chassis -->

Commit message: carlike w wheels wrong

File: description/01_properties.xacro (robot description, xacro)
@@ -23,4 +23,13 @@
     <color rgba="1 1 1 1" />
   </material>
+  <material name="Invisible">
+    <color rgba="0.0 0.0 0.0 0.0"/>
+  </material>
+  <gazebo reference="virtual_rear_wheel">
+    <material>Gazebo/Invisible</material>
+  </gazebo>
+  <gazebo reference="virtual_front_wheel">
+    <material>Gazebo/Invisible</material>
+  </gazebo>
     <!-- Link1 -->
   <gazebo reference="chassis">
@@ -28,23 +37,23 @@
   </gazebo>
   <!-- Link2 -->
-  <gazebo reference="left_wheel">
-    <mu1>0.1</mu1>
-    <mu2>0.1</mu2>
+  <gazebo reference="rear_right_wheel">
+    <mu1>0.01</mu1>
+    <mu2>0.01</mu2>
     <material>Gazebo/Black</material>
   </gazebo>
   <!-- Link3 -->
-  <gazebo reference="right_wheel">
-    <mu1>0.1</mu1>
-    <mu2>0.1</mu2>
+  <gazebo reference="rear_left_wheel">
+    <mu1>0.01</mu1>
+    <mu2>0.01</mu2>
     <material>Gazebo/Black</material>
   </gazebo>
-  <gazebo reference="steering_link">
-    <mu1>0.1</mu1>
-    <mu2>0.1</mu2>
+  <gazebo reference="front_right_wheel">
+    <mu1>0.01</mu1>
+    <mu2>0.01</mu2>
     <material>Gazebo/Black</material>
   </gazebo>
-  <gazebo reference="wheel_front_link">
-    <mu1>0.1</mu1>
-    <mu2>0.1</mu2>
+  <gazebo reference="front_left_wheel">
+    <mu1>0.01</mu1>
+    <mu2>0.01</mu2>
     <material>Gazebo/Black</material>
   </gazebo>

File: description/03_bicycle_drive.xacro (robot description, xacro)
@@ -8,5 +8,5 @@
       <origin xyz="0 0 0" rpy="0 0 0" />
       <geometry>
-        <box size="${base_lx} ${base_ly/4} ${base_lz}" />
+        <box size="${base_lx} ${base_ly} ${base_lz}" />
       </geometry>
     </collision>
@@ -14,5 +14,5 @@
       <origin xyz="0 0 0" rpy="0 0 0" />
       <geometry>
-        <box size="${base_lx} ${base_ly/4} ${base_lz}" />
+        <box size="${base_lx} ${base_ly} ${base_lz}" />
       </geometry>
       <material name="Orange" />
@@ -21,83 +21,175 @@
       <origin xyz="0 0 0" rpy="0 0 0" />
       <mass value="${base_mass}"/>
-      <xacro:box_inertia mass="${base_mass}" width="${base_ly/2}" height="${base_lz}" depth="${base_lx}"/>
+      <xacro:box_inertia mass="${base_mass}" width="${base_ly}" height="${base_lz}" depth="${base_lx}"/>
     </inertial>
   </link>
   <joint name="chassis_joint" type="fixed">
-    <origin xyz="0 0 ${base_lz/2+wheel_radius}" rpy="0 0 0" />
+    <origin xyz="0 0 -${wheel_radius}" rpy="0 0 0" />
     <parent link="base_link" />
     <child link="chassis" />
   </joint>
-  <!-- left wheel Link -->
-  <link name="back_wheel">
+  <link name="virtual_rear_wheel">
+      <visual>
+        <origin xyz="0 0 0" rpy="${PI/2} 0 ${PI/2}"/>
+        <geometry>
+          <cylinder length="0.01" radius="${wheel_radius}"/>
+        </geometry>
+        <material name="Invisible"/>
+      </visual>
+      <inertial>
+        <origin xyz="0 0 0" rpy="0 0 0" />
+        <mass value="0.005" />
+        <inertia ixx="0.001" ixy="0.0" ixz="0.0" iyy="0.001" iyz="0.0" izz="0.001" />
+      </inertial>
+  </link>
+  <joint name="virtual_rear_wheel_joint" type="continuous">
+      <parent link="chassis"/>
+      <child link="virtual_rear_wheel"/>
+      <origin xyz="-${base_lx/2} 0 -${base_lz/2}" rpy="0 0 ${PI/2}"/>
+      <axis xyz="1 0 0"/>
+      <limit effort="100.0" velocity="100.0"/>
+      <dynamics damping="0.02"/>
+  </joint>
+  <!-- right wheel Link -->
+  <link name="rear_right_wheel">
     <collision>
       <geometry>
-        <cylinder length="${wheel_len*4}" radius="${wheel_radius}" />
+        <cylinder length="${wheel_len}" radius="${wheel_radius}" />
       </geometry>
+      <origin xyz="0 0 0" rpy="${PI/2} 0 ${PI/2}"/>
     </collision>
     <visual>
+      <origin xyz="0 0 0" rpy="${PI/2} 0 ${PI/2}"/>
       <geometry>
-        <cylinder length="${wheel_len*4}" radius="${wheel_radius}" />
+        <cylinder length="${wheel_len}" radius="${wheel_radius}" />
       </geometry>
       <material name="Black" />
     </visual>
     <inertial>
+      <origin xyz="0 0 0" rpy="${PI/2} 0 ${PI/2}"/>
+      <mass value="${wheel_mass}" />
+      <xacro:cylinder_inertia mass="${wheel_mass}" radius="${wheel_radius}" height="${wheel_len}"/>
+    </inertial>
+  </link>
+  <joint name="rear_right_wheel_joint" type="continuous">
+    <origin xyz="-${base_lx/2} ${base_ly/2} ${base_lz/2}" rpy="0 0 ${PI/2}" />
+    <parent link="chassis" />
+    <child link="rear_right_wheel" />
+    <axis xyz="1 0 0" />
+    <dynamics damping="0.02" />
+    <limit effort="100.0" velocity="100.0"/>
+    <mimic joint="virtual_rear_wheel_joint" multiplier="1.0" offset="0.0"/>
+  </joint>
+  <!-- left wheel Link -->
+  <link name="rear_left_wheel">
+    <collision>
+      <geometry>
+        <cylinder length="${wheel_len}" radius="${wheel_radius}" />
+      </geometry>
+      <origin xyz="0 0 0" rpy="${PI/2} 0 ${PI/2}"/>
+    </collision>
+    <visual>
+      <origin xyz="0 0 0" rpy="${PI/2} 0 ${PI/2}"/>
+      <geometry>
+        <cylinder length="${wheel_len}" radius="${wheel_radius}" />
+      </geometry>
+      <material name="Black" />
+    </visual>
+    <inertial>
+      <origin xyz="0 0 0" rpy="${PI/2} 0 ${PI/2}"/>
+      <mass value="${wheel_mass}" />
+      <xacro:cylinder_inertia mass="${wheel_mass}" radius="${wheel_radius}" height="${wheel_len}"/>
+    </inertial>
+  </link>
+  <joint name="rear_left_wheel_joint" type="continuous">
+    <origin xyz="-${base_lx/2} -${base_ly/2} ${base_lz/2}" rpy="0 0 ${PI/2}" />
+    <parent link="chassis" />
+    <child link="rear_left_wheel" />
+    <axis xyz="1 0 0" />
+    <dynamics damping="0.02" />
+    <limit effort="100.0" velocity="100.0"/>
+    <mimic joint="virtual_rear_wheel_joint" multiplier="1.0" offset="0.0"/>
+  </joint>
+  <link name="virtual_front_wheel">
+    <visual>
+      <origin xyz="0 0 0" rpy="${PI/2} 0 ${PI/2}"/>
+      <geometry>
+        <cylinder length="0.01" radius="${wheel_radius}"/>
+      </geometry>
+      <material name="Invisible"/>
+    </visual>
+      <inertial>
+        <origin xyz="0 0 0" rpy="0 0 0" />
+        <mass value="0.005" />
+        <inertia ixx="0.001" ixy="0.0" ixz="0.0" iyy="0.001" iyz="0.0" izz="0.001" />
+      </inertial>
+  </link>
+  <joint name="virtual_front_wheel_joint" type="revolute">
+    <parent link="chassis"/>
+    <child link="virtual_front_wheel"/>
+    <origin xyz="${base_lx/2} 0 -${base_lz/2}" rpy="0 0 ${PI/2}"/>
+    <axis xyz="0 0 1"/>
+    <limit lower="-0.8" upper="0.8" effort="100.0" velocity="0.0"/>
+    <dynamics damping="0.02"/>
+  </joint>
+ <!-- right wheel Link -->
+  <link name="front_right_wheel">
+    <collision>
+      <origin xyz="0 0 0" rpy="${PI/2} 0 ${PI/2}"/>
+      <geometry>
+        <cylinder length="${wheel_len}" radius="${wheel_radius}" />
+      </geometry>
+    </collision>
+    <visual>
+     <origin xyz="0 0 0" rpy="${PI/2} 0 ${PI/2}"/>
+      <geometry>
+        <cylinder length="${wheel_len}" radius="${wheel_radius}" />
+      </geometry>
+      <material name="Black" />
+    </visual>
+    <inertial>
+      <origin xyz="0 0 0" rpy="${PI/2} 0 ${PI/2}"/>
       <mass value="${wheel_mass}" />
       <xacro:cylinder_inertia mass="${wheel_mass}" radius="${wheel_radius}" height="${wheel_len*4}"/>
     </inertial>
   </link>
-  <joint name="back_wheel_joint" type="continuous">
-    <origin xyz="-${base_lx/2} 0 ${wheel_radius}" rpy="-1.57 0 0" />
-    <parent link="base_link" />
-    <child link="back_wheel" />
-    <axis xyz="0 0 1" />
-    <dynamics damping="0.2" />
+  <joint name="front_right_wheel_joint" type="revolute">
+    <parent link="chassis" />
+    <child link="front_right_wheel" />
+    <origin xyz="${base_lx/2} ${base_ly/2} -${base_lz/2}" rpy="0 0 ${PI/2}"/>
+    <axis xyz="0 0 1"/>
+    <limit lower="-0.8" upper="0.8" effort="100.0" velocity="0.0"/>
+    <dynamics damping="0.02"/>
+    <mimic joint="virtual_front_wheel_joint" multiplier="1.0" offset="0.0"/>
   </joint>
-    <!-- Steering Link -->
-  <link name="front_steering_link">
+ <!-- left wheel Link -->
+  <link name="front_left_wheel">
+    <collision>
+    <origin xyz="0 0 0" rpy="${PI/2} 0 ${PI/2}"/>
+      <geometry>
+        <cylinder length="${wheel_len}" radius="${wheel_radius}" />
+      </geometry>
+    </collision>
     <visual>
+     <origin xyz="0 0 0" rpy="${PI/2} 0 ${PI/2}"/>
       <geometry>
-        <box size="0.01 0.01 0.01" />
+        <cylinder length="${wheel_len}" radius="${wheel_radius}" />
       </geometry>
       <material name="Black" />
     </visual>
     <inertial>
-      <origin xyz="0 0 0" rpy="0 0 0" />
-      <mass value="0.005" />
-      <inertia ixx="0.1" ixy="0.0" ixz="0.0" iyy="0.1" iyz="0.0" izz="0.1" />
-    </inertial>
-  </link>
-  <joint name="front_steering_joint" type="revolute">
-    <origin xyz="${base_lx/2} 0 ${wheel_radius}" rpy="0 0 0" />
-    <parent link="base_link" />
-    <child link="front_steering_link" />
-    <axis xyz="0 0 1" />
-    <limit effort="100.0" lower="-0.785398" upper="0.785398" velocity="0.1"/>
-  </joint>
-  <!-- right wheel Link -->
-  <link name="front_wheel">
-    <collision>
-      <geometry>
-        <cylinder length="${wheel_len*4}" radius="${wheel_radius}" />
-      </geometry>
-    </collision>
-    <visual>
-      <geometry>
-        <cylinder length="${wheel_len*4}" radius="${wheel_radius}" />
-      </geometry>
-      <material name="Black" />
-    </visual>
-    <inertial>
+      <origin xyz="0 0 0" rpy="${PI/2} 0 ${PI/2}"/>
       <mass value="${wheel_mass}" />
       <xacro:cylinder_inertia mass="${wheel_mass}" radius="${wheel_radius}" height="${wheel_len*4}"/>
     </inertial>
   </link>
-  <joint name="front_wheel_joint" type="continuous">
-    <mimic joint="back_wheel_joint"/>
-    <origin xyz="0 0 0" rpy="-1.57 0 0" />
-    <parent link="front_steering_link" />
-    <child link="front_wheel" />
-    <axis xyz="0 0 1" />
-    <dynamics damping="0.2" />
+  <joint name="front_left_wheel_joint" type="revolute">
+    <parent link="chassis" />
+    <child link="front_left_wheel" />
+    <origin xyz="${base_lx/2} -${base_ly/2} -${base_lz/2}" rpy="0 0 ${PI/2}"/>
+    <axis xyz="0 0 1"/>
+    <limit lower="-0.8" upper="0.8" effort="100.0" velocity="0.0"/>
+    <dynamics damping="0.02"/>
+    <mimic joint="virtual_front_wheel_joint" multiplier="1.0" offset="0.0"/>
   </joint>
 </robot>

File: description/04_bicycle_ros2_control.xacro (robot description, xacro)
@@ -5,5 +5,5 @@
       <plugin>gazebo_ros2_control/GazeboSystem</plugin>
     </hardware>
-    <joint name="back_wheel_joint">
+    <joint name="virtual_rear_wheel_joint">
         <param name="min">-1.0</param>
         <param name="max">1.0</param>
@@ -12,16 +12,33 @@
       <state_interface name="position" />
     </joint>
-    <joint name="front_wheel_joint">
-        <param name="mimic">back_wheel_joint</param>
-        <param name="multiplier">1</param>
-        <param name="min">-1.0</param>
-        <param name="max">1.0</param>
-      <command_interface name="velocity"/>
+    <joint name="rear_right_wheel_joint">
+      <param name="mimic">virtual_rear_wheel_joint</param>
+      <param name="multiplier">1</param>
+      <command_interface name="velocity" />
       <state_interface name="velocity" />
       <state_interface name="position" />
     </joint>
-    <joint name="front_steering_joint">
+    <joint name="rear_left_wheel_joint">
+      <param name="mimic">virtual_rear_wheel_joint</param>
+      <param name="multiplier">1</param>
+      <command_interface name="velocity" />
+      <state_interface name="velocity" />
+      <state_interface name="position" />
+    </joint>
+    <joint name="virtual_front_wheel_joint">
         <param name="min">-0.785</param>
         <param name="max">0.785</param>
+      <command_interface name="position" />
+      <state_interface name="position" />
+    </joint>
+    <joint name="front_right_wheel_joint">
+      <param name="mimic">virtual_front_wheel_joint</param>
+      <param name="multiplier">1</param>
+      <command_interface name="position" />
+      <state_interface name="position" />
+    </joint>
+    <joint name="front_left_wheel_joint">
+      <param name="mimic">virtual_front_wheel_joint</param>
+      <param name="multiplier">1</param>
       <command_interface name="position" />
       <state_interface name="position" />
